Commit message: nav2

File: src/rosbot_description/urdf/rosbot.xacro (robot description, xacro)
@@ -4,4 +4,5 @@
 <xacro:include filename="$(find rosbot_description)/urdf/rosbot.ros2control" />
 <xacro:include filename="$(find rosbot_description)/urdf/rosbot.gazebo" />
+<link name="base_footprint"/>
 <link name="base_link">
   <inertial>
@@ -66,10 +67,10 @@
 <link name="lidar_1">
   <inertial>
-    <origin xyz="0.0 0.0 0.009999999999999981" rpy="0 0 0"/>
+    <origin xyz="0.0 0.0 0.010000000000000009" rpy="0 0 0"/>
     <mass value="0.0754575997873079"/>
     <inertia ixx="1.9e-05" iyy="1.9e-05" izz="3.3e-05" ixy="0.0" iyz="0.0" ixz="0.0"/>
   </inertial>
   <visual>
-    <origin xyz="-0.05 -0.0 -0.12" rpy="0 0 0"/>
+    <origin xyz="-0.05 -0.0 -0.21" rpy="0 0 0"/>
     <geometry>
       <mesh filename="file://$(find rosbot_description)/meshes/lidar_1.stl" scale="0.001 0.001 0.001"/>
@@ -78,5 +79,5 @@
   </visual>
   <collision>
-    <origin xyz="-0.05 -0.0 -0.12" rpy="0 0 0"/>
+    <origin xyz="-0.05 -0.0 -0.21" rpy="0 0 0"/>
     <geometry>
       <mesh filename="file://$(find rosbot_description)/meshes/lidar_1.stl" scale="0.001 0.001 0.001"/>
@@ -84,9 +85,14 @@
   </collision>
 </link>
+<joint name="base_joint" type="fixed">
+  <origin xyz="0.0 0.0 0.0" rpy="0 0 0"/>
+  <parent link="base_footprint"/>
+  <child link="base_link"/>
+</joint>
 <joint name="right_wheel_joint" type="continuous">
   <origin xyz="0.0 -0.1 0.05" rpy="0 0 0"/>
   <parent link="base_link"/>
   <child link="right_wheel_1"/>
-  <axis xyz="0.0 -1.0 0.0"/>
+  <axis xyz="0.0 1.0 0.0"/>
 </joint>
 <joint name="left_wheel_joint" type="continuous">
@@ -97,5 +103,5 @@
 </joint>
 <joint name="lidar_joint" type="fixed">
-  <origin xyz="0.05 0.0 0.12" rpy="0 0 0"/>
+  <origin xyz="0.05 0.0 0.21" rpy="0 0 0"/>
   <parent link="base_link"/>
   <child link="lidar_1"/>
